Commit message: debug for bin-picking

File: urdf/ur10_bin_sim.urdf.xacro (robot description, xacro)
@@ -5,4 +5,5 @@
   <!-- common stuff -->
   <xacro:include filename="$(find agimus_demos)/urdf/ur10_gazebo.xacro" />
+  <xacro:include filename="$(find agimus_demos)/urdf/additional.xacro" />
   <!-- ur10 -->
   <xacro:include filename="$(find ur_description)/urdf/ur10e.xacro" />
@@ -17,163 +18,3 @@
     <xacro:property name="camera_orientation_p" value="${-0.5*M_PI + 0.38}" />
     <xacro:property name="camera_orientation_y" value="0.0" />
-   <!-- Offset of the tip link (obtained by calibration) -->
-   <xacro:arg name="tip_offset_x" default="0.0008"/>
-   <xacro:arg name="tip_offset_y" default="0.0069"/>
-   <xacro:arg name="tip_offset_z" default="0.24"/>
-   <link name="wall_link">
-     <collision>
-       <origin xyz="0 0 1.5"/>
-       <geometry>
-	       <box size="0.1 3 3"/>
-       </geometry>
-     </collision>
-   </link>
-   <joint name="wall_joint" type="fixed">
-     <parent link="world" />
-     <child link = "wall_link" />
-     <origin xyz="-1.4 0.0 0.0" rpy="0.0 0.0 0.0" />
-   </joint>
-    <link name="support_link">
-      <inertial>
-        <mass value="200"/>
-        <origin xyz="0 0 0.3"/>
-        <inertia ixx="50"  ixy="0"  ixz="0" iyy="50" iyz="0" izz="50" />
-      </inertial>
-      <visual>
-        <origin xyz="-0.4 0 0.3"/>
-        <geometry>
-	        <box size="1.0 1.2 0.6"/>
-        </geometry>
-      </visual>
-      <collision>
-        <origin xyz="-0.4 0 0.3"/>
-        <geometry>
-	        <box size="1.0 1.2 0.6"/>
-        </geometry>
-      </collision>
-    </link>
-    <joint name="support_joint" type="fixed">
-      <parent link="world" />
-      <child link = "support_link" />
-      <origin xyz="0.0 0.0 0.0" rpy="0.0 0.0 0.0" />
-    </joint>
-    <joint name="robot_joint" type="fixed">
-      <parent link="support_link" />
-      <child link = "base_link" />
-      <origin xyz="0.0 0.0 0.60" rpy="0.0 0.0 -1.5707963" />
-    </joint>
-    <joint name="ee_fixed_joint" type="fixed">
-     <parent link="wrist_3_link" />
-     <child link = "ee_link" />
-     <origin xyz="0.0 0.0 0.0" rpy="0.0 0.0 ${pi/2.0}" />
-   </joint>
-   <link name="ee_link">
-     <!-- <collision>
-       <geometry>
-         <box size="0.01 0.01 0.01"/>
-       </geometry>
-       <origin rpy="0 0 0" xyz="-0.01 0 0"/>
-     </collision>
-     <visual>
-       <geometry>
-         <box size="0.01 0.01 0.01"/>
-       </geometry>
-       <origin rpy="0 0 0" xyz="-0.01 0 0"/>
-     </visual> -->
-   </link>
-   <link name="ur10e_d435_mount_link">
-     <inertial>
-       <origin xyz="0.0 0.0 0.0" rpy="0 0 0" />
-       <mass value="0.1"/>
-       <inertia ixx="0.001" ixy="0.0" ixz="0.0"
-         iyy="0.001" iyz="0.0"
-         izz="0.001" />
-     </inertial>
-     <visual>
-       <origin xyz="0 0 0" rpy="0 0 0" />
-       <geometry>
-         <mesh filename="package://agimus_demos/meshes/ur10e_d435_mount.stl"/>
-       </geometry>
-       <material name="Red">
-         <color rgba="0.9 0.1 0.1 1.0"/>
-       </material>
-     </visual>
-     <collision>
-       <origin xyz="0 0 0" rpy="0 0 0" />
-       <geometry>
-         <mesh filename="package://agimus_demos/meshes/ur10e_d435_mount.stl"/>
-       </geometry>
-     </collision>
-   </link>
-   <joint name="ur10e_d435_mount_joint" type="fixed">
-     <parent link="wrist_3_link"/>
-     <child link="ur10e_d435_mount_link" />
-     <origin xyz="0.0 0.0 0.0" rpy="0.0 0.0 3.14159265359" />
-   </joint>
-   <link name="ur10e_tool_link">
-     <inertial>
-       <origin xyz="0.0 0.0 0.0" rpy="0 0 0" />
-       <mass value="0.1"/>
-       <inertia ixx="0.001" ixy="0.0" ixz="0.0"
-         iyy="0.001" iyz="0.0"
-         izz="0.001" />
-     </inertial>
-     <!-- Tool support -->
-     <visual>
-       <origin xyz="0 0 0" rpy="0 3.14159265359 0" />
-       <geometry>
-         <mesh filename="package://agimus_demos/meshes/gripper00.stl"/>
-       </geometry>
-       <material name="Red">
-         <color rgba="0.9 0.1 0.1 1.0"/>
-       </material>
-     </visual>
-     <collision>
-       <origin xyz="0 0 0" rpy="0 3.14159265359 0" />
-       <geometry>
-         <mesh filename="package://agimus_demos/meshes/gripper00.stl"/>
-       </geometry>
-     </collision>
-     <!-- wooden spike -->
-     <!--<visual>
-       <origin xyz="0 0 0.113" rpy="0 0 0" />
-       <geometry>
-	 <cylinder radius="0.0015" length="0.25"/>
-       </geometry>
-       <material name="Pine">
-	 <color rgba="0.8 0.65 0.4 1.0"/>
-       </material>
-     </visual>
-     <collision>
-       <origin xyz="0 0 0.113" rpy="0 0 0" />
-       <geometry>
-	 <cylinder radius="0.0015" length="0.25"/>
-       </geometry>
-     </collision>-->
-   </link>
-   <joint name="ur10e_tool_joint" type="fixed">
-     <parent link="ur10e_d435_mount_link"/>
-     <child link="ur10e_tool_link" />
-     <origin xyz="$(arg tip_offset_x) $(arg tip_offset_y) 0.0" rpy="0.0 0.0 0.0" />
-   </joint>
-   <link name="ur10e_tooltip_link">
-   </link>
-  <joint name="ur10e_tooltip_joint" type="fixed">
-     <parent link="ur10e_tool_link" />
-     <child link = "ur10e_tooltip_link" />
-     <origin xyz="0.0 0.0 ${0.25 + $(arg tip_offset_z)}" rpy="0.0 0.0 0.0" />
-  </joint>
-   <link name="ref_camera_link">
-   </link>
-    <joint name="ref_camera_joint" type="fixed">
-     <parent link="ur10e_d435_mount_link" />
-     <child link = "ref_camera_link" />
-     <origin xyz="0.00033351  0.11805402 -0.01064025"
-	     rpy="-0.00127120646 -1.00435876 -1.56137241"/>
-   </joint>
-   <xacro:include filename="$(find realsense2_description)/urdf/_d435.urdf.xacro" />
-   <xacro:sensor_d435 parent="ref_camera_link" name="camera" use_nominal_extrinsics="true">
-     <!-- <origin xyz="0 0.115 0" rpy="0 -1.0472 -1.57079632679"/> -->
-      <origin xyz="0 0 0" rpy="0 0 0"/>
-   </xacro:sensor_d435>
 </robot>
